File: stm32 blue pill.kicad_sch (KiCad schematic)
At the start: 15 parts

Commit message: Power and USB
Power and USB
Parts:
- added C? (x2): 22u, symbol Device:C
- added D?: GREEN, symbol Device:LED
- added J?: Conn_01x04_Male, symbol Connector:Conn_01x04_Male
- added J?: USB_B_Micro, symbol Connector:USB_B_Micro
- added R? (x2): 1k5, symbol Device:R
- added U?: AMS1117-3.3, Package_TO_SOT_SMD:SOT-223-3_TabPin2, symbol Regulator_Linear:AMS1117-3.3
Connections:
- net +3.3V: now also C?.1, D?.2 (A), J?.1 (Pin_1), R?.1, U?.2 (VO)
- net GND: now also C?.2, C?.2, J?.4 (Pin_4), J?.5 (GND), R?.2, U?.1 (GND)
- net SWCLK: now also J?.3 (Pin_3)
- net SWDIO: now also J?.2 (Pin_2)
- net USB_D+: now also J?.3 (D+), R?.2
- net USB_D-: now also J?.2 (D-)
- new net PWR_LED_K: D?.1 (K), R?.1
- new net VBUS: C?.1, J?.1 (VBUS), U?.3 (VI)
- no-connect marks 0 -> 2
Other:
- moved on the sheet: C?, FB?, R?, SW?, U?, Y?

Commit message: schematic updates & pcb init
Parts:
- added C10: 100n, Capacitor_SMD:C_0402_1005Metric, symbol Device:C
- added J1, J2: Conn_01x04_Male, Connector_PinHeader_2.00mm:PinHeader_1x04_P2.00mm_Vertical, symbol Connector:Conn_01x04_Male
- added RP_SCL1, RP_SDA1: 2k2, Resistor_SMD:R_0402_1005Metric, symbol Device:R
- C1, C2: renamed from C?; footprint (none) -> Capacitor_SMD:C_0805_2012Metric
- C11, C12, C13, C3, C4, C5, C7, C8, C9: renamed from C?; footprint (none) -> Capacitor_SMD:C_0402_1005Metric
- C6: renamed from C?; footprint (none) -> Capacitor_SMD:C_0603_1608Metric
- D1: renamed from D?; footprint (none) -> LED_SMD:LED_0603_1608Metric
- FB1: renamed from FB?; footprint (none) -> Inductor_SMD:L_0603_1608Metric
- J3: renamed from J?; footprint (none) -> Connector_USB:USB_Micro-B_Wuerth_629105150521
- J4: renamed from J?; footprint (none) -> Connector_PinHeader_2.00mm:PinHeader_1x04_P2.00mm_Vertical
- R1, R2, R3: renamed from R?; footprint (none) -> Resistor_SMD:R_0402_1005Metric
- SW1: renamed from SW?; footprint (none) -> Button_Switch_SMD:SW_SPDT_PCM12
- Y1: renamed from Y?; footprint (none) -> Crystal:Crystal_SMD_3225-4Pin_3.2x2.5mm
- gave numbers to parts that had none: 2
Connections:
- net +3.3V: now also C10.1, J1.1 (Pin_1), J2.1 (Pin_1), RP_SCL1.1, RP_SDA1.2
- net GND: now also C10.2, J1.4 (Pin_4), J2.4 (Pin_4)
- net I2C2_SCL: now reaches U2.21 (PB10)
- net I2C2_SCL: now also J2.2 (Pin_2), RP_SCL1.2
- net I2C2_SDA: now reaches U2.22 (PB11)
- net I2C2_SDA: now also J2.3 (Pin_3), RP_SDA1.1
- net USART1_TX: now reaches U2.42 (PB6)
- net USART1_TX: now also J1.2 (Pin_2)
- net USART1_RX: now reaches U2.43 (PB7)
- net USART1_RX: now also J1.3 (Pin_3)
- no-connect marks 2 -> 29
Other:
- note added: "1x 100uF per VDD"
- note added: "CL = 2*(CL0-Cs)=2*(10-5)pF=10pF"
- note added: "MCU & USB"
- note added: "Oscillator"
- note added: "Power Supply"
- note added: "USB AN4879 (also found in MCU DS)"
- note added: "VBUS from USB (norm +5V) Min 22uF inp/out caps"
- title: (none) -> Blue Pill (Minimal)
- moved on the sheet: C1, C11, C12, C13, C2, C3, C4, C5, C6, C7, C8, C9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

Commit message: tidying away
Other:
- added sheet Less wrong Blue Pill schematic (untitled.kicad_sch)
- added sheet gps (gps.kicad_sch)
- note added: "Taken with thanks from https://github.com/Jzuni97/STM32-Blue-Pill This is not the schematic of the Blue Pill boards I have. But it is an approximation."
Changed lines of the file:
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@@
 		)
 	)
+	(text "Taken with thanks from\nhttps://github.com/Jzuni97/STM32-Blue-Pill\n\nThis is not the schematic of the Blue Pill boards I have.\nBut it is an approximation."
+		(exclude_from_sim no)
+		(at 54.864 148.59 0)
+		(effects
+			(font
+				(size 1.27 1.27)
+			)
+			(justify left)
+		)
+	)
 	(text "Analog Power Filtering"
 		(exclude_from_sim no)
@@
 				)
 			)
+		)
+	)
+	(sheet
+		(at 25.4 168.91)
+		(size 24.13 3.81)
+		(fields_autoplaced yes)
+		(stroke
+			(width 0.1524)
+			(type solid)
+		)
+		(fill
+			(color 0 0 0 0.0000)
+		)
+		(property "Sheetname" "Less wrong Blue Pill schematic"
+			(at 25.4 168.1984 0)
+			(effects
+				(font
+					(size 1.27 1.27)
+				)
+				(justify left bottom)
+			)
+		)
+		(property "Sheetfile" "untitled.kicad_sch"
+			(at 25.4 173.3046 0)
+			(effects
+				(font
+					(size 1.27 1.27)
+				)
+				(justify left top)
+			)
+		)
+		(instances
+			(project "stm32 blue pill"
+				(path "/7d8f3a67-a21e-4957-b4f0-becb66090b06"
+					(page "2")
+				)
+			)
+		)
+	)
+	(sheet
+		(at 25.4 179.07)
+		(size 12.7 3.81)
+		(fields_autoplaced yes)
+		(stroke
+			(width 0.1524)
+			(type solid)
+		)
+		(fill
+			(color 0 0 0 0.0000)
+		)
+		(property "Sheetname" "gps"
+			(at 25.4 178.3584 0)
+			(effects
+				(font
+					(size 1.27 1.27)
+				)
+				(justify left bottom)
+			)
+		)
+		(property "Sheetfile" "gps.kicad_sch"
+			(at 25.4 183.4646 0)
+			(effects
+				(font
+					(size 1.27 1.27)
+				)
+				(justify left top)
+			)
+		)
+		(instances
+			(project "stm32 blue pill"
+				(path "/7d8f3a67-a21e-4957-b4f0-becb66090b06"
+					(page "3")
+				)
+			)
